File: kicad/EX-PCB-10108-001_connector.sch (KiCad schematic (older format))
At the start: 60 parts, among them CN1 PV-EC-CON-008-014, CN2 PV-EC-CON-013-006, CN3 PV-EC-CON-008-014, CN4 PV-EC-CON-010-010, CN5 PV-EC-CON-012-003, CN6 PV-EC-CON-010-004, U2 PV-EC-PTN-004-004, U3 PV-EC-PTN-004-001, U7 PV-EC-PTN-004-001, U8 PV-EC-PTN-004-001

Commit message: routed power path controller
Parts:
- added J1: Conn_02x02_Odd_Even, Connector_PinHeader_2.54mm:PinHeader_2x02_P2.54mm_Vertical, symbol Connector_Generic:Conn_02x02_Odd_Even
Connections:
- net labels added: ~{LED.GREEN}, ~{LED.RED}, ~{ONOFF}
- net labels removed: ~LED.GREEN, ~LED.RED, ~ONOFF
- wire segments 267 -> 273
Other:
- moved on the sheet: C1, C18, C19, C5, FB1
